File: promicro_smol.kicad_pcb (KiCad board)
At the start: 2 copper layers, 15.2 x 33 mm, 31 parts, among them Q1 HL3134KT, Q2 HL3134KT, Q3 HL3134KT, Q4 HL3134KT, Q5 HL3134KT, U1 LSM6DSVTR, U2 QMC6309, U4 ProMicro NRF52840

Commit message: fix: filenames, minor routing
Routing:
- net GND: track 4.04 -> 3.12 mm
Changed lines of the file:
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@@
 		)
 		(sheetname "/")
-		(sheetfile "promicro_pack.kicad_sch")
+		(sheetfile "promicro_smol.kicad_sch")
 		(attr smd)
 		(fp_line
@@
 		)
 		(sheetname "/")
-		(sheetfile "promicro_pack.kicad_sch")
+		(sheetfile "promicro_smol.kicad_sch")
 		(attr smd)
 		(fp_line
@@
 		)
 		(sheetname "/")
-		(sheetfile "promicro_pack.kicad_sch")
+		(sheetfile "promicro_smol.kicad_sch")
 		(attr through_hole)
 		(fp_line
@@
 		(property ki_fp_filters "C_*")
 		(sheetname "/")
-		(sheetfile "promicro_pack.kicad_sch")
+		(sheetfile "promicro_smol.kicad_sch")
 		(solder_mask_margin 0.038)
 		(attr smd)
@@
 		(property ki_fp_filters "R_*")
 		(sheetname "/")
-		(sheetfile "promicro_pack.kicad_sch")
+		(sheetfile "promicro_smol.kicad_sch")
 		(solder_mask_margin 0.038)
 		(fp_line
@@
 		(property ki_fp_filters "R_*")
 		(sheetname "/")
-		(sheetfile "promicro_pack.kicad_sch")
+		(sheetfile "promicro_smol.kicad_sch")
 		(solder_mask_margin 0.038)
 		(attr smd)
@@
 		)
 		(sheetname "/")
-		(sheetfile "promicro_pack.kicad_sch")
+		(sheetfile "promicro_smol.kicad_sch")
 		(attr smd)
 		(fp_line
@@
 		)
 		(sheetname "/")
-		(sheetfile "promicro_pack.kicad_sch")
+		(sheetfile "promicro_smol.kicad_sch")
 		(attr smd)
 		(fp_line
@@
 		)
 		(sheetname "/")
-		(sheetfile "promicro_pack.kicad_sch")
+		(sheetfile "promicro_smol.kicad_sch")
 		(attr smd)
 		(fp_line
@@
 		(property ki_fp_filters "R_*")
 		(sheetname "/")
-		(sheetfile "promicro_pack.kicad_sch")
+		(sheetfile "promicro_smol.kicad_sch")
 		(solder_mask_margin 0.038)
 		(attr smd)
@@
 		(property ki_fp_filters "R_*")
 		(sheetname "/")
-		(sheetfile "promicro_pack.kicad_sch")
+		(sheetfile "promicro_smol.kicad_sch")
 		(solder_mask_margin 0.038)
 		(fp_line
@@
 		)
 		(sheetname "/")
-		(sheetfile "promicro_pack.kicad_sch")
+		(sheetfile "promicro_smol.kicad_sch")
 		(attr smd)
 		(fp_line
@@
 		(property ki_fp_filters "C_*")
 		(sheetname "/")
-		(sheetfile "promicro_pack.kicad_sch")
+		(sheetfile "promicro_smol.kicad_sch")
 		(solder_mask_margin 0.038)
 		(attr smd)
@@
 		(property ki_fp_filters "R_*")
 		(sheetname "/")
-		(sheetfile "promicro_pack.kicad_sch")
+		(sheetfile "promicro_smol.kicad_sch")
 		(solder_mask_margin 0.038)
 		(fp_line
@@
 		(property ki_fp_filters "R_*")
 		(sheetname "/")
-		(sheetfile "promicro_pack.kicad_sch")
+		(sheetfile "promicro_smol.kicad_sch")
 		(solder_mask_margin 0.038)
 		(fp_line
@@
 		(property ki_fp_filters "R_*")
 		(sheetname "/")
-		(sheetfile "promicro_pack.kicad_sch")
+		(sheetfile "promicro_smol.kicad_sch")
 		(solder_mask_margin 0.038)
 		(fp_line
@@
 		(property ki_fp_filters "R_*")
 		(sheetname "/")
-		(sheetfile "promicro_pack.kicad_sch")
+		(sheetfile "promicro_smol.kicad_sch")
 		(solder_mask_margin 0.038)
 		(fp_line
@@
 		(property ki_fp_filters "R_*")
 		(sheetname "/")
-		(sheetfile "promicro_pack.kicad_sch")
+		(sheetfile "promicro_smol.kicad_sch")
 		(solder_mask_margin 0.038)
 		(fp_line
@@
 		(property ki_fp_filters "R_*")
 		(sheetname "/")
-		(sheetfile "promicro_pack.kicad_sch")
+		(sheetfile "promicro_smol.kicad_sch")
 		(solder_mask_margin 0.038)
 		(fp_line
@@
 		(property ki_fp_filters "C_*")
 		(sheetname "/")
-		(sheetfile "promicro_pack.kicad_sch")
+		(sheetfile "promicro_smol.kicad_sch")
 		(solder_mask_margin 0.038)
 		(attr smd)
@@
 		)
 		(sheetname "/")
-		(sheetfile "promicro_pack.kicad_sch")
+		(sheetfile "promicro_smol.kicad_sch")
 		(attr smd)
 		(fp_line
@@
 		)
 		(sheetname "/")
-		(sheetfile "promicro_pack.kicad_sch")
+		(sheetfile "promicro_smol.kicad_sch")
 		(attr smd exclude_from_pos_files exclude_from_bom allow_missing_courtyard)
 		(fp_rect
@@
 		)
 		(sheetname "/")
-		(sheetfile "promicro_pack.kicad_sch")
+		(sheetfile "promicro_smol.kicad_sch")
 		(attr smd)
 		(fp_line
@@
 		(property ki_fp_filters "R_*")
 		(sheetname "/")
-		(sheetfile "promicro_pack.kicad_sch")
+		(sheetfile "promicro_smol.kicad_sch")
 		(solder_mask_margin 0.038)
 		(fp_line
@@
 		)
 		(sheetname "/")
-		(sheetfile "promicro_pack.kicad_sch")
+		(sheetfile "promicro_smol.kicad_sch")
 		(attr smd)
 		(fp_line
@@
 		(property ki_fp_filters "R_*")
 		(sheetname "/")
-		(sheetfile "promicro_pack.kicad_sch")
+		(sheetfile "promicro_smol.kicad_sch")
 		(solder_mask_margin 0.038)
 		(fp_line
@@
 		(property ki_fp_filters "R_*")
 		(sheetname "/")
-		(sheetfile "promicro_pack.kicad_sch")
+		(sheetfile "promicro_smol.kicad_sch")
 		(solder_mask_margin 0.038)
 		(fp_line
@@
 		(property ki_fp_filters "R_*")
 		(sheetname "/")
-		(sheetfile "promicro_pack.kicad_sch")
+		(sheetfile "promicro_smol.kicad_sch")
 		(solder_mask_margin 0.038)
 		(fp_line
@@
 		(property ki_fp_filters "C_*")
 		(sheetname "/")
-		(sheetfile "promicro_pack.kicad_sch")
+		(sheetfile "promicro_smol.kicad_sch")
 		(solder_mask_margin 0.038)
 		(attr smd)
@@
 		(property ki_fp_filters "R_*")
 		(sheetname "/")
-		(sheetfile "promicro_pack.kicad_sch")
+		(sheetfile "promicro_smol.kicad_sch")
 		(solder_mask_margin 0.038)
 		(fp_line
@@
 		)
 		(sheetname "/")
-		(sheetfile "promicro_pack.kicad_sch")
+		(sheetfile "promicro_smol.kicad_sch")
 		(attr smd)
 		(fp_line
@@
 	)
 	(segment
-		(start 147.6675 117.6025)
-		(end 147.6675 118.4325)
-		(width 0.15)
+		(start 147.4 118.5)
+		(end 147.5 118.6)
+		(width 0.3)
 		(layer "F.Cu")
 		(net 1)
@@
 	)
 	(segment
-		(start 147.1675 117.6025)
-		(end 147.6675 117.6025)
-		(width 0.15)
+		(start 147.4 117.6025)
+		(end 147.4 118.5)
+		(width 0.3)
 		(layer "F.Cu")
 		(net 1)
 	)
 	(segment
-		(start 147.5 117.935)
-		(end 147.1675 117.6025)
-		(width 0.15)
+		(start 147.1675 117.6025)
+		(end 147.4 117.6025)
+		(width 0.3)
 		(layer "F.Cu")
 		(net 1)
@@
 	)
 	(segment
-		(start 147.5 118.6)
-		(end 147.5 117.935)
-		(width 0.15)
+		(start 147.4 117.6025)
+		(end 147.6675 117.6025)
+		(width 0.3)
 		(layer "F.Cu")
 		(net 1)
